File: Rosco-IDE-DRAM/Rosco-IDE-DRAM.kicad_pcb (KiCad board)
At the start: 4 copper layers, 80 x 100 mm, 19 parts, among them J1 Conn_02x05_Odd_Even, J2 Conn_02x22_Odd_Even, U1 74ACT245, U2 74ACT245, U3 ATF1504, U4 74ACT244

Commit message: Mothballing
Parts:
- removed C5: 100nF, Capacitor_SMD:C_0805_2012Metric_Pad1.18x1.45mm_HandSolder
- removed JP1, JP2: SolderJumper_2_Bridged, Jumper:SolderJumper-2_P1.3mm_Bridged_RoundedPad1.0x1.5mm
- removed JP3: SolderJumper_2_Open, Jumper:SolderJumper-2_P1.3mm_Open_RoundedPad1.0x1.5mm
- removed U4: 74ACT244, Package_SO:SOIC-20W_7.5x12.8mm_P1.27mm
- added R2: 4K7, Resistor_THT:R_Axial_DIN0207_L6.3mm_D2.5mm_P7.62mm_Horizontal, F.Cu at (133.2, 84.4)
- added R3: 4K7, Resistor_THT:R_Axial_DIN0207_L6.3mm_D2.5mm_P7.62mm_Horizontal, F.Cu at (133.1, 81.3)
- C1, C2, C3, C4: footprint Capacitor_SMD:C_0805_2012Metric_Pad1.18x1.45mm_HandSolder -> Capacitor_THT:C_Disc_D5.0mm_W2.5mm_P2.50mm
- D1: footprint LED_SMD:LED_0805_2012Metric_Pad1.15x1.40mm_HandSolder -> LED_THT:LED_D5.0mm
- R1: footprint Resistor_SMD:R_0805_2012Metric_Pad1.20x1.40mm_HandSolder -> Resistor_THT:R_Axial_DIN0207_L6.3mm_D2.5mm_P7.62mm_Horizontal
- U1, U2: footprint Package_SO:SOIC-20W_7.5x12.8mm_P1.27mm -> Package_DIP:DIP-20_W7.62mm_LongPads
- moved JP4 80.3 mm to (127.6, 132.2), turned to 90 degrees
- moved J1 64.9 mm to (129.5, 114.5), turned to 0 degrees
- moved C4 61.0 mm to (155.8, 46.5), turned to -90 degrees
- moved C2 59.2 mm to (172.7, 64.1), turned to 180 degrees
- moved U1 53.5 mm to (165.0, 67.7), turned to 0 degrees
- moved R1 42.0 mm to (125.6, 87.6)
- moved D1 33.7 mm to (139.0, 87.7), turned to 180 degrees
- moved C3 27.8 mm to (155.7, 56.6), turned to -90 degrees
- moved U3 26.8 mm to (150.8, 59.0)
- moved J2 26.3 mm to (150.3, 128.2), turned to 180 degrees
- moved U2 7.04 mm to (165.3, 107.8), turned to 0 degrees
- moved C1 3.98 mm to (173.1, 104.6), turned to 180 degrees
- moved SIMM72 2.25 mm to (111.3, 85.1)
Connections:
- net IO64 renamed IDECS_n
- net ~{BRESET} renamed ~{RESET}
- D1 pad 1: GND -> ~{DASP}
- J2 pad 27: unconnected-(J2-Pin_27-Pad27) -> Net-(J2-Pin_27)
- J2 pad 33: BA1 -> A2
- J2 pad 35: BA0 -> A1
- J2 pad 36: BA2 -> A3
- J2 pad 37: ~{CS1} -> ~{CS0}
- J2 pad 38: +5V -> ~{CS1}
- R1 pad 1: ~{DASP} -> +5V
- SIMM72 pad 2: BD0 -> D0
- SIMM72 pad 20: BD4 -> D4
- SIMM72 pad 21: BD4 -> D4
- SIMM72 pad 22: BD5 -> D5
- SIMM72 pad 23: BD5 -> D5
- SIMM72 pad 24: BD6 -> D6
- SIMM72 pad 25: BD6 -> D6
- SIMM72 pad 26: BD7 -> D7
- SIMM72 pad 27: BD7 -> D7
- SIMM72 pad 3: BD0 -> D0
- SIMM72 pad 4: BD1 -> D1
- SIMM72 pad 49: BD8 -> D8
- SIMM72 pad 5: BD1 -> D1
- SIMM72 pad 50: BD8 -> D8
- SIMM72 pad 51: BD9 -> D9
- SIMM72 pad 52: BD9 -> D9
- SIMM72 pad 53: BD10 -> D10
- SIMM72 pad 54: BD10 -> D10
- SIMM72 pad 55: BD11 -> D11
- SIMM72 pad 56: BD11 -> D11
- SIMM72 pad 57: BD12 -> D12
- SIMM72 pad 58: BD12 -> D12
- SIMM72 pad 6: BD2 -> D2
- SIMM72 pad 60: BD13 -> D13
- SIMM72 pad 61: BD13 -> D13
- SIMM72 pad 62: BD14 -> D14
- SIMM72 pad 63: BD14 -> D14
- SIMM72 pad 64: BD15 -> D15
- SIMM72 pad 65: BD15 -> D15
- SIMM72 pad 7: BD2 -> D2
- SIMM72 pad 8: BD3 -> D3
- SIMM72 pad 9: BD3 -> D3
- U1 pad 11: BD7 -> D8
- U1 pad 12: BD6 -> D9
- U1 pad 13: BD5 -> D10
- U1 pad 14: BD4 -> D11
- U1 pad 15: BD3 -> D12
- U1 pad 16: BD2 -> D13
- U1 pad 17: BD1 -> D14
- U1 pad 18: BD0 -> D15
- U1 pad 19: LSEL -> IDEBUF
- U1 pad 2: D0 -> BD7
- U1 pad 3: D1 -> BD6
- U1 pad 4: D2 -> BD5
- U1 pad 5: D3 -> BD4
- U1 pad 6: D4 -> BD3
- U1 pad 7: D5 -> BD2
- U1 pad 8: D6 -> BD1
- U1 pad 9: D7 -> BD0
- U2 pad 11: BD15 -> D0
- U2 pad 12: BD14 -> D1
- U2 pad 13: BD13 -> D2
- U2 pad 14: BD12 -> D3
- U2 pad 15: BD11 -> D4
- U2 pad 16: BD10 -> D5
- U2 pad 17: BD9 -> D6
- U2 pad 18: BD8 -> D7
- U2 pad 19: USEL -> IDEBUF
- U2 pad 2: D8 -> BD15
- U2 pad 3: D9 -> BD14
- U2 pad 4: D10 -> BD13
- U2 pad 5: D11 -> BD12
- U2 pad 6: D12 -> BD11
- U2 pad 7: D13 -> BD10
- U2 pad 8: D14 -> BD9
- U2 pad 9: D15 -> BD8
- U3 pad 10: A17 -> A22
- U3 pad 11: A16 -> A21
- U3 pad 12: A15 -> A20
- U3 pad 15: A14 -> A19
- U3 pad 16: A13 -> A18
- U3 pad 17: A12 -> A17
- U3 pad 18: A11 -> A16
- U3 pad 20: A10 -> A15
- U3 pad 21: A9 -> A14
- U3 pad 22: A8 -> A13
- U3 pad 24: A7 -> A12
- U3 pad 25: A6 -> A11
- U3 pad 27: A5 -> A10
- U3 pad 28: A4 -> A9
- U3 pad 29: A3 -> A8
- U3 pad 30: A2 -> A7
- U3 pad 31: A1 -> A6
- U3 pad 33: IOSEL -> A5
- U3 pad 34: EXPSEL -> A4
- U3 pad 35: FC0 -> A3
- U3 pad 36: FC1 -> A2
- U3 pad 37: FC2 -> A1
- U3 pad 39: LDS -> ~{MWE}
- U3 pad 4: A22 -> UDS
- U3 pad 40: UDS -> ~{RAS1}
- U3 pad 41: RW -> ~{RAS0}
- U3 pad 44: DTACK -> ~{CAS1}
- U3 pad 45: LSEL -> ~{CAS3}
- U3 pad 46: USEL -> ~{CAS2}
- U3 pad 48: CS1 -> ~{CAS0}
- U3 pad 49: ~{IDEWR} -> MA8
- U3 pad 5: A21 -> EXPSEL
- U3 pad 50: ~{IDERD} -> MA9
- U3 pad 51: VPA -> MA11
- U3 pad 52: MA0 -> MA7
- U3 pad 54: MA1 -> MA10
- U3 pad 55: MA2 -> MA6
- U3 pad 56: MA3 -> MA5
- U3 pad 58: MA5 -> MA3
- U3 pad 6: A20 -> IOSEL
- U3 pad 60: MA6 -> MA2
- U3 pad 61: MA7 -> MA1
- U3 pad 63: MA8 -> MA0
- U3 pad 64: MA9 -> unconnected-(U3-I/O-Pad64)
- U3 pad 65: MA10 -> unconnected-(U3-I/O-Pad65)
- U3 pad 67: MA11 -> unconnected-(U3-I/O-Pad67)
- U3 pad 68: ~{RAS0} -> ~{IDEWR}
- U3 pad 69: ~{RAS1} -> ~{IDERD}
- U3 pad 70: ~{CAS0} -> RW
- U3 pad 73: ~{CAS1} -> IDEBUF
- U3 pad 74: ~{CAS2} -> CS0
- U3 pad 75: ~{CAS3} -> CS1
- U3 pad 76: ~{MWE} -> DTACK
- U3 pad 79: IO65 -> FC2
- U3 pad 8: A19 -> VPA
- U3 pad 80: IO66 -> FC1
- U3 pad 81: GCLK3/IO -> FC0
- U3 pad 9: A18 -> A23
Routing:
- net IDEBUF: track 0.00 -> 139.7 mm
- net BD14: track 120.5 -> 13.5 mm, vias 1 -> 0
- net GND: track 101.4 -> 0.00 mm, vias 15 -> 0
- net BD13: track 110.6 -> 13.3 mm, vias 1 -> 0
- net BD12: track 110.3 -> 13.1 mm, vias 1 -> 0
- net D12: track 17.8 -> 111.2 mm, vias 0 -> 1
- net LSEL: track 91.2 -> 0.00 mm, vias 1 -> 0
- net D11: track 18.5 -> 107.9 mm
- net BD15: track 102.4 -> 13.8 mm, vias 1 -> 0
- net D13: track 18.3 -> 104.1 mm, vias 0 -> 2
- net ~{CAS2}: track 105.8 -> 23.9 mm, vias 0 -> 1
- net D14: track 19.0 -> 96.7 mm
- net D10: track 19.0 -> 96.0 mm
- net D9: track 19.5 -> 96.3 mm
- net BD11: track 89.0 -> 13.1 mm, vias 1 -> 0
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Other:
- board text added: "Rosco-IDE-DRAM, Malcolm Harrow, December 2024, v2"
- board text removed: "Rosco-IDE-DRAM, Malcolm Harrow, April 2024, v1"
