File: Rosco-IDE-DRAM/Rosco-IDE-DRAM.kicad_sch (KiCad schematic)
At the start: 19 parts, among them J1 Conn_02x05_Odd_Even, J2 Conn_02x22_Odd_Even, U1 74ACT245, U2 74ACT245, U3 ATF1504, U4 74ACT244

Commit message: Mothballing
Parts:
- removed JP1, JP2: SolderJumper_2_Bridged, Jumper:SolderJumper-2_P1.3mm_Bridged_RoundedPad1.0x1.5mm, symbol Jumper:SolderJumper_2_Bridged
- removed JP3: SolderJumper_2_Open, Jumper:SolderJumper-2_P1.3mm_Open_RoundedPad1.0x1.5mm, symbol Jumper:SolderJumper_2_Open
- removed U4: 74ACT244, Package_SO:SOIC-20W_7.5x12.8mm_P1.27mm, symbol 74xx:74HCT244
- added C6: 100nF, Capacitor_THT:C_Disc_D5.0mm_W2.5mm_P2.50mm, symbol Device:C
- added IC1, IC2: ATF22V10C-15PU, Package_DIP:DIP-24_18.0mmx34.29mm_W15.24mm_LongPads, symbol ATF22V10:ATF22V10C-15PU
- added R2, R3: 4K7, Resistor_THT:R_Axial_DIN0207_L6.3mm_D2.5mm_P7.62mm_Horizontal, symbol Device:R
- C1, C2, C3, C4, C5: footprint Capacitor_SMD:C_0805_2012Metric_Pad1.18x1.45mm_HandSolder -> Capacitor_THT:C_Disc_D5.0mm_W2.5mm_P2.50mm
- D1: footprint LED_SMD:LED_0805_2012Metric_Pad1.15x1.40mm_HandSolder -> LED_THT:LED_D5.0mm
- R1: footprint Resistor_SMD:R_0805_2012Metric_Pad1.20x1.40mm_HandSolder -> Resistor_THT:R_Axial_DIN0207_L6.3mm_D2.5mm_P7.62mm_Horizontal
- U1, U2: footprint Package_SO:SOIC-20W_7.5x12.8mm_P1.27mm -> Package_DIP:DIP-20_W7.62mm_LongPads
Connections:
- net BA0 is gone; now on net A1: J2.35 (Pin_35)
- net BA1 is gone; now on net A2: J2.33 (Pin_33)
- net BA2 is gone; now on net A3: J2.36 (Pin_36)
- net GCLK3/IO is gone; now on net FC0: U3.81 (GCLK3/I/O)
- net IO65 is gone; now on net FC2: U3.79 (I/O)
- net IO66 is gone; now on net FC1: U3.80 (I/O)
- net +5V: now also R1.1, C6.1, IC1.24 (VCC), IC2.24 (VCC); no longer J2.38 (Pin_38)
- net A1: now also U3.37 (I/O), IC2.11 (IN_9); no longer U3.31 (I/O)
- net A10: now also U3.27 (I/O), IC1.15 (I/O_2); no longer U3.20 (PD1/I/O)
- net A11: now also U3.25 (I/O), IC1.14 (I/O_1); no longer U3.18 (I/O)
- net A12: now also U3.24 (I/O), IC1.13 (IN_10); no longer U3.17 (I/O)
- net A13: now also U3.22 (I/O), IC1.11 (IN_9); no longer U3.16 (I/O)
- net A14: now also U3.21 (I/O), IC1.10 (IN_8); no longer U3.15 (I/O)
- net A15: now also U3.20 (PD1/I/O), IC1.9 (IN_7); no longer U3.12 (I/O)
- net A16: now also U3.18 (I/O), IC1.8 (IN_6); no longer U3.11 (I/O)
- net A17: now also U3.17 (I/O), IC1.7 (IN_5); no longer U3.10 (I/O)
- net A18: now also U3.16 (I/O), IC1.6 (IN_4); no longer U3.9 (I/O)
- net A19: now also U3.15 (I/O), IC1.5 (IN_3); no longer U3.8 (I/O)
- net A2: now also U3.36 (I/O), IC2.10 (IN_8); no longer U3.30 (I/O)
- net A20: now also U3.12 (I/O); no longer U3.6 (I/O)
- net A21: now also U3.11 (I/O); no longer U3.5 (I/O)
- net A22: now also U3.10 (I/O); no longer U3.4 (I/O)
- net A23: now also U3.9 (I/O); no longer U3.3 (VCCINT)
- net A3: now also U3.35 (I/O), IC2.9 (IN_7); no longer U3.29 (I/O)
- net A4: now also U3.34 (I/O), IC2.8 (IN_6); no longer U3.28 (I/O)
- net A5: now also U3.33 (I/O), IC2.7 (IN_5); no longer U3.27 (I/O)
- net A6: now also U3.31 (I/O), IC1.19 (I/O_6); no longer U3.25 (I/O)
- net A7: now also U3.30 (I/O), IC1.18 (I/O_5); no longer U3.24 (I/O)
- net A8: now also U3.29 (I/O), IC1.17 (I/O_4); no longer U3.22 (I/O)
- net A9: now also U3.28 (I/O), IC1.16 (I/O_3); no longer U3.21 (I/O)
- net BD0: now also U1.9 (A7); no longer SIMM72.2 (DQ0), SIMM72.3 (DQ16), U1.18 (B0)
- net BD1: now also U1.8 (A6); no longer SIMM72.4 (DQ1), SIMM72.5 (DQ17), U1.17 (B1)
- net BD10: now also U2.7 (A5); no longer SIMM72.53 (DQ10), SIMM72.54 (DQ26), U2.16 (B2)
- net BD11: now also U2.6 (A4); no longer SIMM72.55 (DQ11), SIMM72.56 (DQ27), U2.15 (B3)
- net BD12: now also U2.5 (A3); no longer SIMM72.57 (DQ12), SIMM72.58 (DQ28), U2.14 (B4)
- net BD13: now also U2.4 (A2); no longer SIMM72.60 (DQ29), SIMM72.61 (DQ13), U2.13 (B5)
- net BD14: now also U2.3 (A1); no longer SIMM72.62 (DQ30), SIMM72.63 (DQ14), U2.12 (B6)
- net BD15: now also U2.2 (A0); no longer SIMM72.64 (DQ31), SIMM72.65 (DQ15), U2.11 (B7)
- net BD2: now also U1.7 (A5); no longer SIMM72.6 (DQ2), SIMM72.7 (DQ18), U1.16 (B2)
- net BD3: now also U1.6 (A4); no longer SIMM72.8 (DQ3), SIMM72.9 (DQ19), U1.15 (B3)
- net BD4: now also U1.5 (A3); no longer SIMM72.20 (DQ4), SIMM72.21 (DQ20), U1.14 (B4)
- net BD5: now also U1.4 (A2); no longer SIMM72.22 (DQ5), SIMM72.23 (DQ21), U1.13 (B5)
- net BD6: now also U1.3 (A1); no longer SIMM72.24 (DQ6), SIMM72.25 (DQ22), U1.12 (B6)
- net BD7: now also U1.2 (A0); no longer SIMM72.26 (DQ7), SIMM72.27 (DQ23), U1.11 (B7)
- net BD8: now also U2.9 (A7); no longer SIMM72.49 (DQ8), SIMM72.50 (DQ24), U2.18 (B0)
- net BD9: now also U2.8 (A6); no longer SIMM72.51 (DQ9), SIMM72.52 (DQ25), U2.17 (B1)
- net CS1: now also U3.75 (I/O); no longer U3.48 (I/O)
- net D0: now also SIMM72.2 (DQ0), SIMM72.3 (DQ16), U2.11 (B7); no longer U1.2 (A0)
- net D1: now also SIMM72.4 (DQ1), SIMM72.5 (DQ17), U2.12 (B6); no longer U1.3 (A1)
- net D10: now also SIMM72.53 (DQ10), SIMM72.54 (DQ26), U1.13 (B5); no longer U2.4 (A2)
- net D11: now also SIMM72.55 (DQ11), SIMM72.56 (DQ27), U1.14 (B4); no longer U2.5 (A3)
- net D12: now also SIMM72.57 (DQ12), SIMM72.58 (DQ28), U1.15 (B3); no longer U2.6 (A4)
- net D13: now also SIMM72.60 (DQ29), SIMM72.61 (DQ13), U1.16 (B2); no longer U2.7 (A5)
- net D14: now also SIMM72.62 (DQ30), SIMM72.63 (DQ14), U1.17 (B1); no longer U2.8 (A6)
- net D15: now also SIMM72.64 (DQ31), SIMM72.65 (DQ15), U1.18 (B0); no longer U2.9 (A7)
- net D2: now also SIMM72.6 (DQ2), SIMM72.7 (DQ18), U2.13 (B5); no longer U1.4 (A2)
- net D3: now also SIMM72.8 (DQ3), SIMM72.9 (DQ19), U2.14 (B4); no longer U1.5 (A3)
- net D4: now also SIMM72.20 (DQ4), SIMM72.21 (DQ20), U2.15 (B3); no longer U1.6 (A4)
- net D5: now also SIMM72.22 (DQ5), SIMM72.23 (DQ21), U2.16 (B2); no longer U1.7 (A5)
- net D6: now also SIMM72.24 (DQ6), SIMM72.25 (DQ22), U2.17 (B1); no longer U1.8 (A6)
- net D7: now also SIMM72.26 (DQ7), SIMM72.27 (DQ23), U2.18 (B0); no longer U1.9 (A7)
- net D8: now also SIMM72.49 (DQ8), SIMM72.50 (DQ24), U1.11 (B7); no longer U2.2 (A0)
- net D9: now also SIMM72.51 (DQ9), SIMM72.52 (DQ25), U1.12 (B6); no longer U2.3 (A1)
- net DTACK: now also U3.76 (I/O); no longer U3.44 (I/O)
- net EXPSEL: now also U3.5 (I/O); no longer U3.34 (I/O)
- net FC0: now also IC1.1 (CLK/IN), IC2.1 (CLK/IN); no longer U3.35 (I/O)
- net FC1: now also IC1.2 (IN_1), IC2.2 (IN_1); no longer U3.36 (I/O)
- net FC2: now also IC1.3 (IN_2), IC2.3 (IN_2); no longer U3.37 (I/O)
- net GND: now also C6.2, IC1.12 (GND), IC2.12 (GND), R2.2, R3.2; no longer D1.1 (K)
- net INTRQ: now also R3.1
- net IOSEL: now also U3.6 (I/O); no longer U3.33 (I/O)
- net LDS: now also U3.3 (VCCINT); no longer U3.39 (I/O)
- net MA0: now also U3.63 (I/O); no longer U3.52 (I/O)
- net MA1: now also U3.61 (I/O); no longer U3.54 (I/O)
- net MA10: now also U3.54 (I/O); no longer U3.65 (I/O)
- net MA11: now also U3.51 (I/O); no longer U3.67 (I/O)
- net MA2: now also U3.60 (I/O); no longer U3.55 (I/O)
- net MA3: now also U3.58 (I/O); no longer U3.56 (I/O)
- net MA5: now also U3.56 (I/O); no longer U3.58 (I/O)
- net MA6: now also U3.55 (I/O); no longer U3.60 (I/O)
- net MA7: now also U3.52 (I/O); no longer U3.61 (I/O)
- net MA8: now also U3.49 (I/O); no longer U3.63 (I/O)
- net MA9: now also U3.50 (I/O); no longer U3.64 (I/O)
- net RW: now also U3.70 (I/O), IC2.4 (IN/PD); no longer U3.41 (I/O)
- net UDS: now also U3.4 (I/O); no longer U3.40 (I/O)
- net VPA: now also U3.8 (I/O), IC2.14 (I/O_1); no longer U3.51 (I/O)
- net ~{CAS0}: now also U3.48 (I/O); no longer U3.70 (I/O)
- net ~{CAS1}: now also U3.44 (I/O); no longer U3.73 (I/O)
- net ~{CAS2}: now also U3.46 (I/O/PD2); no longer U3.74 (I/O)
- net ~{CAS3}: now also U3.45 (I/O); no longer U3.75 (I/O)
- net ~{CS1}: now also J2.38 (Pin_38); no longer J2.37 (Pin_37)
- net ~{DASP}: now also D1.1 (K); no longer R1.1
- net ~{IDERD}: now also U3.69 (I/O), IC2.20 (I/O_7); no longer U3.50 (I/O)
- net ~{IDEWR}: now also U3.68 (I/O), IC2.19 (I/O_6); no longer U3.49 (I/O)
- net ~{MWE}: now also U3.39 (I/O); no longer U3.76 (I/O)
- net ~{RAS0}: now also U3.41 (I/O); no longer U3.68 (I/O)
- net ~{RAS1}: now also U3.40 (I/O); no longer U3.69 (I/O)
- net at J2.27 (Pin_27): now also R2.1
- net IO64 renamed IDECS_n
- net LSEL renamed IDEBUF
- net IDEBUF: now also U2.19 (CE), U3.73 (I/O); no longer U3.45 (I/O)
- removed net USEL: U2.19 (CE), U3.46 (I/O/PD2)
- net ~{BRESET} renamed ~{RESET}
- new net CS0: U3.74 (I/O)
- new net IDESEL: IC2.21 (I/O_8)
- new net ~{AS}: IC2.5 (IN_3)
- new net ~{CS0}: J2.37 (Pin_37)
- new net ~{DTACK}: IC2.17 (I/O_4)
- new net ~{IDEBUF}: IC2.18 (I/O_5)
- new net ~{IDECS0}: IC2.16 (I/O_3)
- new net ~{IDECS1}: IC2.15 (I/O_2)
- new net ~{IDECS}: IC1.23 (I/O_10)
- new net ~{IOSEL}: IC1.4 (IN/PD)
- new net ~{UDS}: IC2.6 (IN_4)
- no-connect marks 30 -> 28
Other:
- note added: "Note the bytes are swapped to convert to 68k endianess"
- note added: "wire CPU_SPACE = (FC0 && FC1 && FC2); assign IDECS_n = !(!CPU_SPACE && !IOSEL_n && (A[19:6] == 13'b10000000000001)); assign IDECS0_n = !(!IDECS_n && !A5 && A4); assign IDECS1_n = !(!IDECS_n && A5 && !A4); assign IDERD_n = !(RW && !AS_n && !UDS_n); assign IDEWR_n = !(!RW && !AS_n && !UDS_n); assign IDEBUF_n = ~(~IDECS0_n || ~IDECS1_n); wire IDE_SELECTED = ~AS_n && (~IDECS0_n || ~IDECS1_n); assign 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"
